Commit message: fix 2th 4-1

File: description/robot.urdf.xacro (robot description, xacro)
@@ -3,5 +3,3 @@
     <!-- Example link -->
     <link name="base_link"></link>
-    <link name="h"></link>
-    <link name="j"></link>
 </robot>

Commit message: fix 1th 8-1

File: description/robot.urdf.xacro (robot description, xacro)
@@ -2,3 +2,4 @@
 <robot xmlns:xacro="http://www.ros.org/wiki/xacro"  name="robot">
     <xacro:include filename="robot_core.xacro"/>
+    <xacro:include filename="gazebo_control.xacro"/>
 </robot>

File: description/robot_core.xacro (robot description, xacro)
@@ -14,8 +14,7 @@
         <color rgba="0.2 0.2 1 1" />
     </material>
-    <xacro:property name="chassis_length" value="2.1" />
     <link name="base_link">
+    </link>
     <!--CHASSIS LINK-->
-    </link>
     <joint name="chassis_joint" type="fixed">
         <parent link="base_link"/>
@@ -25,14 +24,14 @@
     <link name="chassis">
         <visual>
-            <origin xyz="0.125 0 0.033" rpy="0 0 0"/>
+            <origin xyz="0.125 0 0.03" rpy="0 0 0"/>
             <geometry>
-                <box size="0.25 0.2 0.066"/>
+                <box size="0.25 0.2 0.06"/>
             </geometry>
             <material name="white"/>
         </visual>
         <collision>
-            <origin xyz="0.125 0 0.033" rpy="0 0 0"/>
+            <origin xyz="0.125 0 0.03" rpy="0 0 0"/>
             <geometry>
-                <box size="0.25 0.2 0.066"/>
+                <box size="0.25 0.2 0.06"/>
             </geometry>
         </collision>
@@ -41,9 +40,12 @@
         </xacro:inertial_box>
     </link>
+    <gazebo reference="chassis">
+        <material>Gazebo/White</material>
+    </gazebo>
     <!--WHEEL LINK-->
     <joint name="left_wheel_joint" type="continuous">
         <parent link="base_link"/>
         <child link="left_wheel"/>
-        <origin xyz="0 0.1 0" rpy="-${pi/2} 0 0"/>
+        <origin xyz="0 0.113 0" rpy="-${pi/2} 0 0"/>
         <axis xyz="0 0 1"/>
     </joint>
@@ -64,8 +66,11 @@
         </xacro:inertial_cylinder>
     </link>
+    <gazebo reference="left_wheel">
+        <material>Gazebo/Blue</material>
+    </gazebo>
     <joint name="right_wheel_joint" type="continuous">
         <parent link="base_link"/>
         <child link="right_wheel"/>
-        <origin xyz="0 -0.1 0" rpy="${pi/2} 0 0"/>
+        <origin xyz="0 -0.113 0" rpy="${pi/2} 0 0"/>
         <axis xyz="0 0 -1"/>
     </joint>
@@ -86,4 +91,7 @@
         </xacro:inertial_cylinder>
     </link>
+    <gazebo reference="right_wheel">
+        <material>Gazebo/Blue</material>
+    </gazebo>
     <!--CASTER WHEEL LINK-->
     <joint name="caster_wheel_joint" type="fixed">
@@ -108,4 +116,9 @@
         </xacro:inertial_sphere>
     </link>
+    <gazebo reference="caster_wheel">
+        <material>Gazebo/Black</material>
+        <mu1 value="0.001"/>
+        <mu2 value="0.001"/>
+    </gazebo>
     <joint name="caster1_wheel_joint" type="fixed">
         <parent link="chassis"/>
@@ -129,3 +142,8 @@
         </xacro:inertial_sphere>
     </link>
+    <gazebo reference="caster1_wheel">
+        <material>Gazebo/Black</material>
+        <mu1 value="0.001"/>
+        <mu2 value="0.001"/>
+    </gazebo>
 </robot>

Commit message: fix 1st 12-1

File: description/robot.urdf.xacro (robot description, xacro)
@@ -3,3 +3,4 @@
     <xacro:include filename="robot_core.xacro"/>
     <xacro:include filename="gazebo_control.xacro"/>
+    <xacro:include filename="lidar.xacro"/>
 </robot>

File: description/robot_core.xacro (robot description, xacro)
@@ -13,4 +13,7 @@
     <material name="blue">
         <color rgba="0.2 0.2 1 1" />
+    </material>
+    <material name="red">
+        <color rgba="1 0 0 1" />
     </material>
     <link name="base_link">

Commit message: 21-1

File: description/robot.urdf.xacro (robot description, xacro)
@@ -1,7 +1,13 @@
 <?xml version="1.0"?>
 <robot xmlns:xacro="http://www.ros.org/wiki/xacro"  name="robot">
+    <xacro:arg name="use_ros2_control" default="true"/>
+    <xacro:arg name="sim_mode" default="false"/>
     <xacro:include filename="robot_core.xacro"/>
-    <!--<xacro:include filename="gazebo_control.xacro"/> -->
-    <xacro:include filename="ros2_control.xacro"/>
+    <xacro:if value="$(arg use_ros2_control)">
+        <xacro:include filename="ros2_control.xacro" />
+    </xacro:if>
+    <xacro:unless value="$(arg use_ros2_control)">
+        <xacro:include filename="gazebo_control.xacro" />
+    </xacro:unless>
     <xacro:include filename="lidar.xacro"/>
 </robot>

File: description/robot_core.xacro (robot description, xacro)
@@ -62,5 +62,5 @@
         <collision>
             <geometry>
-                <cylinder radius="0.033" length="0.026"/>
+                <sphere radius="0.033"/>
             </geometry>
         </collision>
@@ -87,5 +87,5 @@
         <collision>
             <geometry>
-                <cylinder radius="0.033" length="0.026"/>
+                <sphere radius="0.033"/>
             </geometry>
         </collision>

File: description/ros2_control.xacro (robot description, xacro)
@@ -1,28 +1,59 @@
 <?xml version="1.0"?>
 <robot xmlns:xacro="http://www.ros.org/wiki/xacro">
-    <ros2_control name="GazeboSystem" type="system">
-        <hardware>
-            <plugin>gazebo_ros2_control/GazeboSystem</plugin>
-        </hardware>
-        <joint name="left_wheel_joint">
-            <command_interface name="velocity">
-                <param name="min">-10</param>
-                <param name="max">10</param>
-            </command_interface>
-            <state_interface name="velocity"/>
-            <state_interface name="position"/>
-        </joint>
-        <joint name="right_wheel_joint">
-            <command_interface name="velocity">
-                <param name="min">-10</param>
-                <param name="max">10</param>
-            </command_interface>
-            <state_interface name="velocity"/>
-            <state_interface name="position"/>
-        </joint>
-    </ros2_control>
+    <xacro:unless value="$(arg sim_mode)">
+        <ros2_control name="RealRobot" type="system">
+            <hardware>
+                <plugin>diffdrive_arduino/DiffDriveArduinoHardware</plugin>
+                <param name="left_wheel_name">left_wheel_joint</param>
+                <param name="right_wheel_name">right_wheel_joint</param>
+                <param name="loop_rate">100</param>
+                <param name="device">/dev/ttyUSB0</param>
+                <param name="baud_rate">57600</param>
+                <param name="timeout_ms">1000</param>
+                <param name="enc_counts_per_rev">1540</param>
+                <param name="pid_p">30</param>
+                <param name="pid_d">12</param>
+                <param name="pid_i">0</param>
+                <param name="pid_o">50</param>
+            </hardware>
+            <joint name="left_wheel_joint">
+                <command_interface name="velocity"/>
+                <state_interface name="position"/>
+                <state_interface name="velocity"/>
+            </joint>
+            <joint name="right_wheel_joint">
+                <command_interface name="velocity"/>
+                <state_interface name="position"/>
+                <state_interface name="velocity"/>
+            </joint>
+        </ros2_control>
+    </xacro:unless>
+    <xacro:if value="$(arg sim_mode)">
+        <ros2_control name="GazeboSystem" type="system">
+            <hardware>
+                <plugin>gazebo_ros2_control/GazeboSystem</plugin>
+            </hardware>
+            <joint name="left_wheel_joint">
+                <command_interface name="velocity">
+                    <param name="min">-10</param>
+                    <param name="max">10</param>
+                </command_interface>
+                <state_interface name="velocity"/>
+                <state_interface name="position"/>
+            </joint>
+            <joint name="right_wheel_joint">
+                <command_interface name="velocity">
+                    <param name="min">-10</param>
+                    <param name="max">10</param>
+                </command_interface>
+                <state_interface name="velocity"/>
+                <state_interface name="position"/>
+            </joint>
+        </ros2_control>
+    </xacro:if>
     <gazebo>
         <plugin name="gazebo_ros2_control" filename="libgazebo_ros2_control.so">
             <parameters>$(find my_robot)/config/my_controllers.yaml</parameters>
+            <parameters>$(find my_robot)/config/gaz_use_sim_time.yaml</parameters>
         </plugin>
     </gazebo>
