Commit message: fix on lab 6-1

File: description/robot_core.xacro (robot description, xacro)
@@ -15,3 +15,50 @@
     <link name="base_link">
     </link>
+    <joint name="chassis_joint" type="fixed">
+        <parent link="base_link"/>
+        <child link="chassis"/>
+        <origin xyz="-0.1 0 0"/>
+    </joint>
+    <link name="chassis">
+        <visual>
+            <origin xyz="0.125 0 0.05"/>
+            <geometry>
+                <box size="0.25 0.2 0.1"/>
+            </geometry>
+            <material name="white"/>
+        </visual>
+    </link>
+    <joint name="left_wheel_joint" type="continuous">
+        <parent link="base_link"/>
+        <child link="left_wheel"/>
+        <origin xyz="0 0.1 0" rpy="-${pi/2} 0 0"/>
+        <axis xyz="0 0 1"/>
+    </joint>
+    <link name="left_wheel">
+        <visual>
+            <geometry>
+                <cylinder radius="0.032" length="0.025"/>
+            </geometry>
+        </visual>
+        <material name="blue"/>
+    </link>
+    <joint name="right_wheel_joint" type="continuous">
+        <parent link="base_link"/>
+        <child link="right_wheel"/>
+        <origin xyz="0 -0.1 0" rpy="${pi/2} 0 0"/>
+        <axis xyz="0 0 -1"/>
+    </joint>
+    <link name="right_wheel">
+        <visual>
+            <geometry>
+                <cylinder radius="0.032" length="0.025"/>
+            </geometry>
+        </visual>
+        <material name="blue"/>
+    </link>
+    <joint name="caster_wheel_joint" type="fixed">
+        <parent link="chassis"/>
+        <child link="caster_wheel"/>
+        <origin xyz="0.05 0 "
+    </joint>
 </robot>

Commit message: fix 1th 7-1

File: description/robot_core.xacro (robot description, xacro)
@@ -60,5 +60,5 @@
         <parent link="chassis"/>
         <child link="caster_wheel"/>
-        <origin xyz="0.05 0 "
+        <origin xyz="0.05 0 "/>
     </joint>
 </robot>

Commit message: fix 2th 7-1

File: description/robot_core.xacro (robot description, xacro)
@@ -1,4 +1,5 @@
 <?xml version="1.0"?>
 <robot xmlns:xacro="http://www.ros.org/wiki/xacro" >
+    <xacro:include filename="inertial_macros.xacro"/>
     <material name="white">
         <color rgba="1 1 1 1" />
@@ -13,20 +14,32 @@
         <color rgba="0.2 0.2 1 1" />
     </material>
+    <xacro:property name="chassis_length" value="2.1" />
     <link name="base_link">
+    <!--CHASSIS LINK-->
     </link>
     <joint name="chassis_joint" type="fixed">
         <parent link="base_link"/>
         <child link="chassis"/>
-        <origin xyz="-0.1 0 0"/>
+        <origin xyz="-0.145 0 0"/>
     </joint>
     <link name="chassis">
         <visual>
-            <origin xyz="0.125 0 0.05"/>
+            <origin xyz="0.125 0 0.033" rpy="0 0 0"/>
             <geometry>
-                <box size="0.25 0.2 0.1"/>
+                <box size="0.25 0.2 0.066"/>
             </geometry>
             <material name="white"/>
         </visual>
+        <collision>
+            <origin xyz="0.125 0 0.033" rpy="0 0 0"/>
+            <geometry>
+                <box size="0.25 0.2 0.066"/>
+            </geometry>
+        </collision>
+        <xacro:inertial_box mass="2.0" x="0.25" y="0.2" z="0.066">
+            <origin xyz="0.125 0 0.033"/>
+        </xacro:inertial_box>
     </link>
+    <!--WHEEL LINK-->
     <joint name="left_wheel_joint" type="continuous">
         <parent link="base_link"/>
@@ -38,8 +51,16 @@
         <visual>
             <geometry>
-                <cylinder radius="0.032" length="0.025"/>
+                <cylinder radius="0.033" length="0.026"/>
             </geometry>
+            <material name="blue"/>
         </visual>
-        <material name="blue"/>
+        <collision>
+            <geometry>
+                <cylinder radius="0.033" length="0.026"/>
+            </geometry>
+        </collision>
+        <xacro:inertial_cylinder mass="0.05" length="0.026" radius="0.033">
+            <origin xyz="0 0 0" rpy="0 0 0"/>
+        </xacro:inertial_cylinder>
     </link>
     <joint name="right_wheel_joint" type="continuous">
@@ -52,13 +73,59 @@
         <visual>
             <geometry>
-                <cylinder radius="0.032" length="0.025"/>
+                <cylinder radius="0.033" length="0.026"/>
             </geometry>
+            <material name="blue"/>
         </visual>
-        <material name="blue"/>
+        <collision>
+            <geometry>
+                <cylinder radius="0.033" length="0.026"/>
+            </geometry>
+        </collision>
+        <xacro:inertial_cylinder mass="0.05" length="0.026" radius="0.033">
+            <origin xyz="0 0 0" rpy="0 0 0"/>
+        </xacro:inertial_cylinder>
     </link>
+    <!--CASTER WHEEL LINK-->
     <joint name="caster_wheel_joint" type="fixed">
         <parent link="chassis"/>
         <child link="caster_wheel"/>
-        <origin xyz="0.05 0 "/>
+        <origin xyz="0.05 0 -0.0185"/>
     </joint>
+    <link name="caster_wheel">
+        <visual>
+            <geometry>
+                <sphere radius="0.0145"/>
+            </geometry>
+            <material name="black"/>
+        </visual>
+        <collision>
+            <geometry>
+                <sphere radius="0.0145"/>
+            </geometry>
+        </collision>
+        <xacro:inertial_sphere mass="0.01" radius="0.0145">
+            <origin xyz="0 0 0" rpy="0 0 0"/>
+        </xacro:inertial_sphere>
+    </link>
+    <joint name="caster1_wheel_joint" type="fixed">
+        <parent link="chassis"/>
+        <child link="caster1_wheel"/>
+        <origin xyz="0.24 0 -0.0255"/>
+    </joint>
+    <link name="caster1_wheel">
+        <visual>
+            <geometry>
+                <sphere radius="0.0075"/>
+            </geometry>
+            <material name="black"/>
+        </visual>
+        <collision>
+            <geometry>
+                <sphere radius="0.0075"/>
+            </geometry>
+        </collision>
+        <xacro:inertial_sphere mass="0.005" radius="0.0075">
+            <origin xyz="0 0 0" rpy="0 0 0"/>
+        </xacro:inertial_sphere>
+    </link>
 </robot>

Commit message: fix 1st 23-1

File: description/robot_core.xacro (robot description, xacro)
@@ -18,4 +18,11 @@
     </material>
     <link name="base_link">
+    </link>
+    <joint name="base_footprint_joint" type="fixed">
+        <parent link="base_link"/>
+        <child link="base_footprint"/>
+        <origin xyz="0 0 0" rpy="0 0 0"/>
+    </joint>
+    <link name="base_footprint">
     </link>
     <!--CHASSIS LINK-->

Commit message: fist

File: description/robot_core.xacro (robot description, xacro)
@@ -26,134 +26,3 @@
     <link name="base_footprint">
     </link>
-    <!--CHASSIS LINK-->
-    <joint name="chassis_joint" type="fixed">
-        <parent link="base_link"/>
-        <child link="chassis"/>
-        <origin xyz="-0.145 0 0"/>
-    </joint>
-    <link name="chassis">
-        <visual>
-            <origin xyz="0.125 0 0.03" rpy="0 0 0"/>
-            <geometry>
-                <box size="0.25 0.2 0.06"/>
-            </geometry>
-            <material name="white"/>
-        </visual>
-        <collision>
-            <origin xyz="0.125 0 0.03" rpy="0 0 0"/>
-            <geometry>
-                <box size="0.25 0.2 0.06"/>
-            </geometry>
-        </collision>
-        <xacro:inertial_box mass="3.0" x="0.25" y="0.2" z="0.06685">
-            <origin xyz="0.125 0 0.033"/>
-        </xacro:inertial_box>
-    </link>
-    <gazebo reference="chassis">
-        <material>Gazebo/White</material>
-    </gazebo>
-    <!--WHEEL LINK-->
-    <joint name="left_wheel_joint" type="continuous">
-        <parent link="base_link"/>
-        <child link="left_wheel"/>
-        <origin xyz="0 0.113 0" rpy="-${pi/2} 0 0"/>
-        <axis xyz="0 0 1"/>
-    </joint>
-    <link name="left_wheel">
-        <visual>
-            <geometry>
-                <cylinder radius="0.033" length="0.026"/>
-            </geometry>
-            <material name="blue"/>
-        </visual>
-        <collision>
-            <geometry>
-                <sphere radius="0.033"/>
-            </geometry>
-        </collision>
-        <xacro:inertial_cylinder mass="0.05" length="0.026" radius="0.033">
-            <origin xyz="0 0 0" rpy="0 0 0"/>
-        </xacro:inertial_cylinder>
-    </link>
-    <gazebo reference="left_wheel">
-        <material>Gazebo/Blue</material>
-    </gazebo>
-    <joint name="right_wheel_joint" type="continuous">
-        <parent link="base_link"/>
-        <child link="right_wheel"/>
-        <origin xyz="0 -0.113 0" rpy="${pi/2} 0 0"/>
-        <axis xyz="0 0 -1"/>
-    </joint>
-    <link name="right_wheel">
-        <visual>
-            <geometry>
-                <cylinder radius="0.033" length="0.026"/>
-            </geometry>
-            <material name="blue"/>
-        </visual>
-        <collision>
-            <geometry>
-                <sphere radius="0.033"/>
-            </geometry>
-        </collision>
-        <xacro:inertial_cylinder mass="0.05" length="0.026" radius="0.033">
-            <origin xyz="0 0 0" rpy="0 0 0"/>
-        </xacro:inertial_cylinder>
-    </link>
-    <gazebo reference="right_wheel">
-        <material>Gazebo/Blue</material>
-    </gazebo>
-    <!--CASTER WHEEL LINK-->
-    <joint name="caster_wheel_joint" type="fixed">
-        <parent link="chassis"/>
-        <child link="caster_wheel"/>
-        <origin xyz="0.02 0 -0.0185"/>
-    </joint>
-    <link name="caster_wheel">
-        <visual>
-            <geometry>
-                <sphere radius="0.0145"/>
-            </geometry>
-            <material name="black"/>
-        </visual>
-        <collision>
-            <geometry>
-                <sphere radius="0.0145"/>
-            </geometry>
-        </collision>
-        <xacro:inertial_sphere mass="0.01" radius="0.0145">
-            <origin xyz="0 0 0" rpy="0 0 0"/>
-        </xacro:inertial_sphere>
-    </link>
-    <gazebo reference="caster_wheel">
-        <material>Gazebo/Black</material>
-        <mu1 value="0.001"/>
-        <mu2 value="0.001"/>
-    </gazebo>
-    <joint name="caster1_wheel_joint" type="fixed">
-        <parent link="chassis"/>
-        <child link="caster1_wheel"/>
-        <origin xyz="0.24 0 -0.0255"/>
-    </joint>
-    <link name="caster1_wheel">
-        <visual>
-            <geometry>
-                <sphere radius="0.0075"/>
-            </geometry>
-            <material name="black"/>
-        </visual>
-        <collision>
-            <geometry>
-                <sphere radius="0.0075"/>
-            </geometry>
-        </collision>
-        <xacro:inertial_sphere mass="0.005" radius="0.0075">
-            <origin xyz="0 0 0" rpy="0 0 0"/>
-        </xacro:inertial_sphere>
-    </link>
-    <gazebo reference="caster1_wheel">
-        <material>Gazebo/Black</material>
-        <mu1 value="0.001"/>
-        <mu2 value="0.001"/>
-    </gazebo>
 </robot>
