Commit message: fix 25-1

File: description/lidar.xacro (robot description, xacro)
@@ -18,5 +18,5 @@
             </geometry>
         </collision>
-        <xacro:inertial_cylinder mass="0.1" length="0.03" radius="0.032">
+        <xacro:inertial_cylinder mass="0.25" length="0.03" radius="0.032">
             <origin xyz="0 0 0" rpy="0 0 0"/>
         </xacro:inertial_cylinder>

File: description/robot_core.xacro (robot description, xacro)
@@ -46,5 +46,5 @@
             </geometry>
         </collision>
-        <xacro:inertial_box mass="2.0" x="0.25" y="0.2" z="0.066">
+        <xacro:inertial_box mass="3.0" x="0.25" y="0.2" z="0.06685">
             <origin xyz="0.125 0 0.033"/>
         </xacro:inertial_box>
@@ -108,5 +108,5 @@
         <parent link="chassis"/>
         <child link="caster_wheel"/>
-        <origin xyz="0.05 0 -0.0185"/>
+        <origin xyz="0.02 0 -0.0185"/>
     </joint>
     <link name="caster_wheel">

File: description/ros2_control.xacro (robot description, xacro)
@@ -8,8 +8,8 @@
                 <param name="right_wheel_name">right_wheel_joint</param>
                 <param name="loop_rate">100</param>
-                <param name="device">/dev/ttyUSB0</param>
+                <param name="device">/dev/ttyUSB1</param>
                 <param name="baud_rate">57600</param>
                 <param name="timeout_ms">1000</param>
-                <param name="enc_counts_per_rev">1540</param>
+                <param name="enc_counts_per_rev">1457</param>
                 <param name="pid_p">30</param>
                 <param name="pid_d">12</param>

Commit message: fix 25-1

File: description/lidar.xacro (robot description, xacro)
@@ -2,5 +2,5 @@
 <robot xmlns:xacro="http://www.ros.org/wiki/xacro" >
     <joint name="laser_joint" type="fixed">
-        <parent link="chassis"/>
+        <parent link="chassis_link"/>
         <child link="laser_frame"/>
         <origin xyz="0.097 0 0.14" rpy="0 0 0"/>
@@ -11,5 +11,5 @@
                 <cylinder radius="0.032" length="0.03"/>
             </geometry>
-            <material name="black"/>
+            <material name="green"/>
         </visual>
         <collision>
@@ -18,10 +18,10 @@
             </geometry>
         </collision>
-        <xacro:inertial_cylinder mass="0.25" length="0.03" radius="0.032">
+        <xacro:inertial_cylinder mass="0.3" length="0.03" radius="0.032">
             <origin xyz="0 0 0" rpy="0 0 0"/>
         </xacro:inertial_cylinder>
     </link>
     <gazebo reference="laser_frame">
-        <material>Gazebo/Red</material>
+        <material>Gazebo/Green</material>
         <sensor name="laser" type="ray">
             <pose> 0 0 0 0 0 0 </pose>

File: description/robot_core.xacro (robot description, xacro)
@@ -12,11 +12,37 @@
     </material>
     <material name="blue">
-        <color rgba="0.2 0.2 1 1" />
+        <color rgba="0.1764 0.4588 0.8509 1.0" />
     </material>
     <material name="red">
         <color rgba="1 0 0 1" />
     </material>
+    <material name="yellow">
+        <color rgba="0.8784 0.6627 0.6627 1.0"/>
+    </material>
+    <material name="green">
+        <color rgba="0.003 0.639 0.223 1.0"/>
+    </material>
+    <xacro:property name="chassis_length" value="0.25"/>
+    <xacro:property name="chassis_width" value="0.2"/>
+    <xacro:property name="chassis_height" value="0.06685"/>
+    <xacro:property name="chassis_mass" value="3.0"/>
+    <xacro:property name="wheel_radius" value="0.033"/>
+    <xacro:property name="wheel_thickness" value="0.026"/>
+    <xacro:property name="wheel_mass" value="0.05"/>
+    <xacro:property name="wheel_offset_x" value="0.125"/>
+    <xacro:property name="wheel_offset_y" value="0.123"/>
+    <xacro:property name="wheel_offset_z" value="0"/>
+    <xacro:property name="caster_wheel_radius" value="0.0125"/>
+    <xacro:property name="caster_wheel_mass" value="0.01"/>
+    <xacro:property name="caster_wheel_offset_x" value="0.02"/>
+    <xacro:property name="caster_wheel_offset_z" value="${wheel_offset_z - wheel_radius + caster_wheel_radius}"/>
+    <xacro:property name="front_caster_wheel_radius" value="0.0075"/>
+    <xacro:property name="front_caster_wheel_mass" value="0.01"/>
+    <xacro:property name="front_caster_wheel_offset_x" value="0.24"/>
+    <xacro:property name="front_caster_wheel_offset_z" value="${wheel_offset_z - wheel_radius + front_caster_wheel_radius}"/>
+    <!-- BASE LINK -->
     <link name="base_link">
     </link>
+    <!-- BASE_FOOTPRINT LINK -->
     <joint name="base_footprint_joint" type="fixed">
         <parent link="base_link"/>
@@ -26,3 +52,135 @@
     <link name="base_footprint">
     </link>
+    <!-- CHASSIS LINK -->
+    <joint name="chassis_joint" type="fixed">
+        <parent link="base_link"/>
+        <child link="chassis_link"/>
+        <origin xyz="-${wheel_offset_x} 0 ${wheel_offset_z}"/>
+    </joint>
+    <link name="chassis_link">
+        <visual>
+            <origin xyz="${chassis_length/2} 0 ${chassis_height/2}"/>
+            <geometry>
+                <box size="${chassis_length} ${chassis_width} ${chassis_height}"/>
+            </geometry>
+            <material name="white"/>
+        </visual>
+        <collision>
+            <origin xyz="${chassis_length/2} 0 ${chassis_height/2}"/>
+            <geometry>
+                <box size="${chassis_length} ${chassis_width} ${chassis_height}"/>
+            </geometry>
+        </collision>
+        <xacro:inertial_box mass="${chassis_mass}" x="${chassis_length}" y="${chassis_width}" z="${chassis_height}">
+          <origin xyz="${chassis_length/2} 0 ${chassis_height/2}" rpy="0 0 0"/>
+        </xacro:inertial_box>
+    </link>
+    <gazebo reference="chassis_link">
+      <material>Gazebo/White</material>
+    </gazebo>
+    <!-- RIGHT WHEEL -->
+    <joint name="right_wheel_joint" type="continuous">
+        <parent link="base_link"/>
+        <child link="right_wheel_link"/>
+        <origin xyz="0 -${wheel_offset_y} ${wheel_offset_z}" rpy="${pi/2} 0 0" />
+        <axis xyz="0 0 -1"/>
+    </joint>
+    <link name="right_wheel_link">
+        <visual>
+            <geometry>
+                <cylinder radius="${wheel_radius}" length="${wheel_thickness}"/>
+            </geometry>
+            <material name="blue"/>
+        </visual>
+        <collision>
+            <geometry>
+                <sphere radius="${wheel_radius}"/>
+            </geometry>
+        </collision>
+        <xacro:inertial_cylinder mass="${wheel_mass}" length="${wheel_thickness}" radius="${wheel_radius}">
+          <origin xyz="0 0 0" rpy="0 0 0"/>
+        </xacro:inertial_cylinder>
+    </link>
+    <gazebo reference="right_wheel_link">
+      <material>Gazebo/Blue</material>
+    </gazebo>
+    <!-- LEFT WHEEL -->
+    <joint name="left_wheel_joint" type="continuous">
+        <parent link="base_link"/>
+        <child link="left_wheel_link"/>
+        <origin xyz="0 ${wheel_offset_y} ${wheel_offset_z}" rpy="-${pi/2} 0 0" />
+        <axis xyz="0 0 1"/>
+    </joint>
+    <link name="left_wheel_link">
+        <visual>
+            <geometry>
+                <cylinder radius="${wheel_radius}" length="${wheel_thickness}"/>
+            </geometry>
+            <material name="blue"/>
+        </visual>
+        <collision>
+            <geometry>
+                <sphere radius="${wheel_radius}"/>
+            </geometry>
+        </collision>
+        <xacro:inertial_cylinder mass="${wheel_mass}" length="${wheel_thickness}" radius="${wheel_radius}">
+            <origin xyz="0 0 0" rpy="0 0 0"/>
+        </xacro:inertial_cylinder>
+    </link>
+    <gazebo reference="left_wheel_link">
+      <material>Gazebo/Blue</material>
+    </gazebo>
+    <!-- CASTER WHEEL LINK -->
+    <joint name="caster_wheel_joint" type="fixed">
+        <parent link="chassis_link"/>
+        <child link="caster_wheel"/>
+        <origin xyz="${caster_wheel_offset_x} 0 ${caster_wheel_offset_z}"/>
+    </joint>
+    <link name="caster_wheel">
+        <visual>
+            <geometry>
+                <sphere radius="${caster_wheel_radius}"/>
+            </geometry>
+            <material name="black"/>
+        </visual>
+        <collision>
+            <geometry>
+                <sphere radius="${caster_wheel_radius}"/>
+            </geometry>
+        </collision>
+        <xacro:inertial_sphere mass="${caster_wheel_mass}" radius="${caster_wheel_radius}">
+            <origin xyz="0 0 0" rpy="0 0 0"/>
+        </xacro:inertial_sphere>
+    </link>
+    <gazebo reference="caster_wheel">
+        <material>Gazebo/Black</material>
+        <mu1 value="0.001"/>
+        <mu2 value="0.001"/>
+    </gazebo>
+    <joint name="front_caster_wheel_joint" type="fixed">
+        <parent link="chassis_link"/>
+        <child link="front_caster_wheel"/>
+        <origin xyz="${front_caster_wheel_offset_x} 0 ${front_caster_wheel_offset_z}"/>
+    </joint>
+    <link name="front_caster_wheel">
+        <visual>
+            <geometry>
+                <sphere radius="${front_caster_wheel_radius}"/>
+            </geometry>
+            <material name="black"/>
+        </visual>
+        <collision>
+            <geometry>
+                <sphere radius="${front_caster_wheel_radius}"/>
+            </geometry>
+        </collision>
+        <xacro:inertial_sphere mass="${front_caster_wheel_mass}" radius="${front_caster_wheel_radius}">
+            <origin xyz="0 0 0" rpy="0 0 0"/>
+        </xacro:inertial_sphere>
+    </link>
+    <gazebo reference="front_caster_wheel">
+        <material>Gazebo/Black</material>
+        <mu1 value="0.001"/>
+        <mu2 value="0.001"/>
+    </gazebo>
 </robot>

File: description/ros2_control.xacro (robot description, xacro)
@@ -13,7 +13,7 @@
                 <param name="enc_counts_per_rev">1457</param>
                 <param name="pid_p">30</param>
-                <param name="pid_d">12</param>
+                <param name="pid_d">20</param>
                 <param name="pid_i">0</param>
-                <param name="pid_o">50</param>
+                <param name="pid_o">100</param>
             </hardware>
             <joint name="left_wheel_joint">
